File: canhat.kicad_sch (KiCad schematic)
At the start: 41 parts, among them J1 Raspberry_Pi_2_3, J2 CAN In/Out/GND, J3 GPIO, J5 12V, U1 MCP2515-xSO, U2 SN65HVDA541, U3 AT24C32-SSHM, U4 AP63205, Y1 16MHz

Commit message: Replaced resistors with solder bridges
Parts:
- removed R10: DNP/0, Resistor_SMD:R_0805_2012Metric_Pad1.20x1.40mm_HandSolder, symbol Device:R
- removed R6: DNP, Resistor_SMD:R_0805_2012Metric_Pad1.20x1.40mm_HandSolder, symbol Device:R
- removed R7: 0, Resistor_SMD:R_0805_2012Metric_Pad1.20x1.40mm_HandSolder, symbol Device:R
- added JP2: IOCTL, Jumper:SolderJumper-3_P1.3mm_Bridged12_RoundedPad1.0x1.5mm_NumberLabels, symbol Jumper:Jumper_3_Bridged12
- added JP3: 3VIO, Jumper:SolderJumper-2_P1.3mm_Bridged_RoundedPad1.0x1.5mm, symbol Jumper:Jumper_2_Bridged
- added JP4: VBUS, Jumper:SolderJumper-3_P1.3mm_Bridged12_RoundedPad1.0x1.5mm_NumberLabels, symbol Jumper:Jumper_3_Bridged12
- added JP5: 5VIN, Jumper:SolderJumper-2_P1.3mm_Open_RoundedPad1.0x1.5mm, symbol Jumper:Jumper_2_Open
- L1: footprint onitake:DS75LC -> Inductor_SMD:L_TDK_SLF7032
- renumbered D7 to D2, F2 to F1
Connections:
- net +12LF: now also JP5.2 (B)
- net +3V3: now also JP3.2 (B), JP4.3 (B)
- net +5V: now also JP4.1 (A), JP5.1 (A); no longer C6.1, U2.3 (VCC)
- net GND: now also C6.1, JP2.1 (A); no longer C6.2, R5.1
- net TRXEN: now also JP2.3 (B)
- net at U2.5 (EN): now also JP3.1 (A)
- net at U2.8 (Rs): now also R5.1; no longer R5.2
- new net: C6.2, JP4.2 (C), U2.3 (VCC)
- new net: JP2.2 (C), R5.2
Other:
- moved on the sheet: C3, C4, C6, C7, J2, U2
